Commit message: add: colors

File: lidar_robot_model/urdf/body/body.urdf.xacro (robot description, xacro)
@@ -13,4 +13,7 @@
           <box size="0.400 0.200 0.100"/>
         </geometry>
+        <material name="gray">
+          <color rgba="1 1 1 1"/>
+        </material>
       </visual>
       <collision>

File: lidar_robot_model/urdf/caster/caster.urdf.xacro (robot description, xacro)
@@ -13,4 +13,7 @@
           <sphere radius="0.05"/>
         </geometry>
+        <material name="green">
+          <color rgba="0 128 0 1"/>
+        </material>
       </visual>
       <collision>

File: lidar_robot_model/urdf/lidar_base/lidar_base.urdf.xacro (robot description, xacro)
@@ -13,4 +13,7 @@
           <box size="0.150 0.150 0.100"/>
         </geometry>
+        <material name="gray">
+          <color rgba="1 1 1 1"/>
+        </material>
       </visual>
       <collision>

File: lidar_robot_model/urdf/wheel/wheel.urdf.xacro (robot description, xacro)
@@ -15,4 +15,7 @@
           <cylinder radius="0.1" length="0.05"/>
         </geometry>
+        <material name="olive">
+          <color rgba="128 128 0 1"/>
+        </material>
       </visual>
       <collision>
